File: leg-controller.kicad_pcb (KiCad board)
At the start: 0 parts

Commit message: Started workin on PCB layout. A bit faulty...
Parts:
- added C1: 470u, Capacitor_THT:CP_Radial_D10.0mm_P5.00mm, F.Cu at (111.8, 119.4)
- added C10: 100n, Capacitor_SMD:C_0603_1608Metric_Pad1.05x0.95mm_HandSolder, F.Cu at (124.4, 64.4)
- added C11: 100n, Capacitor_SMD:C_0603_1608Metric_Pad1.05x0.95mm_HandSolder, F.Cu at (137.5, 48.5)
- added C3: 10u, Capacitor_THT:CP_Radial_D5.0mm_P2.00mm, F.Cu at (123.4, 111.3)
- added C4: 22p, Capacitor_SMD:C_0603_1608Metric_Pad1.05x0.95mm_HandSolder, F.Cu at (141.9, 48.5)
- added C5: 22p, Capacitor_SMD:C_0603_1608Metric_Pad1.05x0.95mm_HandSolder, F.Cu at (130.7, 57.7)
- added C6: 100n, Capacitor_SMD:C_0603_1608Metric_Pad1.05x0.95mm_HandSolder, F.Cu at (137.5, 51.0)
- added C7: 100n, Capacitor_SMD:C_0603_1608Metric_Pad1.05x0.95mm_HandSolder, F.Cu at (136.2, 78.0)
- added C8: 100n, Capacitor_SMD:C_0603_1608Metric_Pad1.05x0.95mm_HandSolder, F.Cu at (109.0, 77.0)
- added C9: 100n, Capacitor_SMD:C_0603_1608Metric_Pad1.05x0.95mm_HandSolder, F.Cu at (167.6, 42.7)
- added D1: D_Schottky_x2_Serial_AKC, Package_TO_SOT_SMD:SOT-323_SC-70, F.Cu at (122.3, 85.9)
- added D10: LED, LED_SMD:LED_0603_1608Metric_Pad1.05x0.95mm_HandSolder, F.Cu at (99.9, 85.3)
- added D11: LED, LED_SMD:LED_0603_1608Metric_Pad1.05x0.95mm_HandSolder, F.Cu at (158.5, 51.0)
- added D2: D_Schottky_x2_Serial_AKC, Package_TO_SOT_SMD:SOT-323_SC-70, F.Cu at (90.8, 85.9)
- added D3: D_Schottky_x2_Serial_AKC, Package_TO_SOT_SMD:SOT-323_SC-70, F.Cu at (149.4, 51.7)
- added D4: LED_POWER, LED_SMD:LED_0603_1608Metric_Pad1.05x0.95mm_HandSolder, F.Cu at (126.3, 56.8)
- added D5: LED_3V3, LED_SMD:LED_0603_1608Metric_Pad1.05x0.95mm_HandSolder, F.Cu at (106.3, 67.3)
- added D6: D, Diode_SMD:D_SOD-123F, F.Cu at (121.4, 117.9)
- added D7: LED_ERR, LED_SMD:LED_0603_1608Metric_Pad1.05x0.95mm_HandSolder, F.Cu at (131.0, 55.1)
- added D8: LED_RUN, LED_SMD:LED_0603_1608Metric_Pad1.05x0.95mm_HandSolder, F.Cu at (126.3, 59.4)
- added D9: LED, LED_SMD:LED_0603_1608Metric_Pad1.05x0.95mm_HandSolder, F.Cu at (131.4, 85.3)
- added J1: Power, TerminalBlock:TerminalBlock_Altech_AK300-2_P5.00mm, F.Cu at (97.5, 119.4)
- added J10: Motor, Connector_PinHeader_2.54mm:PinHeader_1x03_P2.54mm_Vertical, F.Cu at (154.1, 39.9)
- added J11: Rotary_Encoder, Connector_PinHeader_2.54mm:PinHeader_1x04_P2.54mm_Vertical, F.Cu at (149.5, 39.9)
- added J12: UART, Connector_PinHeader_2.54mm:PinHeader_1x04_P2.54mm_Vertical, F.Cu at (95.5, 54.7)
- added J14: ISP, Connector_PinHeader_2.54mm:PinHeader_2x03_P2.54mm_Vertical, F.Cu at (91.4, 96.0)
- added J15: Motor_E, Connector_PinHeader_2.54mm:PinHeader_1x05_P2.54mm_Vertical, F.Cu at (90.9, 39.9)
- added J16: Motor_D, Connector_PinHeader_2.54mm:PinHeader_1x05_P2.54mm_Vertical, F.Cu at (90.9, 54.7)
- added J17: Motor_F, Connector_PinHeader_2.54mm:PinHeader_1x05_P2.54mm_Vertical, F.Cu at (95.5, 39.9)
- added J2: I2C, Connector_PinHeader_2.54mm:PinHeader_1x03_P2.54mm_Vertical, F.Cu at (93.5, 132.6)
- added J3: Conn_02x01, Connector_PinHeader_2.54mm:PinHeader_1x02_P2.54mm_Vertical, F.Cu at (131.7, 79.1)
- added J4: Motor, Connector_PinHeader_2.54mm:PinHeader_1x03_P2.54mm_Vertical, F.Cu at (127.1, 74.2)
- added J5: Rotary_Encoder, Connector_PinHeader_2.54mm:PinHeader_1x04_P2.54mm_Vertical, F.Cu at (122.4, 74.2)
- added J6: Conn_02x01, Connector_PinHeader_2.54mm:PinHeader_1x02_P2.54mm_Vertical, F.Cu at (100.2, 79.1)
- added J7: Motor, Connector_PinHeader_2.54mm:PinHeader_1x03_P2.54mm_Vertical, F.Cu at (95.5, 74.2)
- added J8: Rotary_Encoder, Connector_PinHeader_2.54mm:PinHeader_1x04_P2.54mm_Vertical, F.Cu at (90.9, 74.2)
- added J9: Conn_02x01, Connector_PinHeader_2.54mm:PinHeader_1x02_P2.54mm_Vertical, F.Cu at (158.8, 44.8)
- added NT1: Net-Tie_2, NetTie:NetTie-2_THT_Pad1.0mm, F.Cu at (100.1, 67.4)
- added NT2: Net-Tie_2, NetTie:NetTie-2_THT_Pad1.0mm, F.Cu at (94.6, 67.4)
- added Q1: Q_NPN_BEC, Package_TO_SOT_SMD:SOT-23, F.Cu at (127.0, 83.8)
- added Q3: Q_NPN_BEC, Package_TO_SOT_SMD:SOT-23, F.Cu at (95.4, 83.8)
- added Q5: Q_NPN_BEC, Package_TO_SOT_SMD:SOT-23, F.Cu at (154.0, 49.6)
- added R10: 100, Resistor_SMD:R_0603_1608Metric_Pad1.05x0.95mm_HandSolder, F.Cu at (144.9, 80.7)
- added R11: 330, Resistor_SMD:R_0603_1608Metric_Pad1.05x0.95mm_HandSolder, F.Cu at (144.9, 78.1)
- added R12: 5m, Resistor_SMD:R_2512_6332Metric, F.Cu at (133.7, 74.3)
- added R13: 1k, Resistor_SMD:R_0603_1608Metric_Pad1.05x0.95mm_HandSolder, F.Cu at (112.9, 84.5)
- added R14: 4.7k, Resistor_SMD:R_0603_1608Metric_Pad1.05x0.95mm_HandSolder, F.Cu at (113.4, 80.7)
- added R15: 10k, Resistor_SMD:R_0603_1608Metric_Pad1.05x0.95mm_HandSolder, F.Cu at (113.4, 78.1)
- added R16: 10k, Resistor_SMD:R_0603_1608Metric_Pad1.05x0.95mm_HandSolder, F.Cu at (104.7, 78.0)
- added R17: 5.23k, Resistor_SMD:R_0603_1608Metric_Pad1.05x0.95mm_HandSolder, F.Cu at (108.5, 84.5)
- added R18: 47k, Resistor_SMD:R_0603_1608Metric_Pad1.05x0.95mm_HandSolder, F.Cu at (109.0, 82.0)
- added R19: 10k, Resistor_SMD:R_0603_1608Metric_Pad1.05x0.95mm_HandSolder, F.Cu at (114.5, 75.6)
- added R2: 1k, Resistor_SMD:R_0603_1608Metric_Pad1.05x0.95mm_HandSolder, F.Cu at (146.1, 73.1)
- added R20: 100, Resistor_SMD:R_0603_1608Metric_Pad1.05x0.95mm_HandSolder, F.Cu at (109.0, 79.5)
- added R21: 100, Resistor_SMD:R_0603_1608Metric_Pad1.05x0.95mm_HandSolder, F.Cu at (104.2, 85.2)
- added R22: 330, Resistor_SMD:R_0603_1608Metric_Pad1.05x0.95mm_HandSolder, F.Cu at (114.5, 73.1)
- added R23: 5m, Resistor_SMD:R_2512_6332Metric, F.Cu at (102.2, 74.3)
- added R24: 1k, Resistor_SMD:R_0603_1608Metric_Pad1.05x0.95mm_HandSolder, F.Cu at (167.6, 47.7)
- added R25: 4.7k, Resistor_SMD:R_0603_1608Metric_Pad1.05x0.95mm_HandSolder, F.Cu at (173.2, 46.4)
- added R26: 10k, Resistor_SMD:R_0603_1608Metric_Pad1.05x0.95mm_HandSolder, F.Cu at (167.2, 50.2)
- added R27: 10k, Resistor_SMD:R_0603_1608Metric_Pad1.05x0.95mm_HandSolder, F.Cu at (171.5, 55.3)
- added R28: 5.23k, Resistor_SMD:R_0603_1608Metric_Pad1.05x0.95mm_HandSolder, F.Cu at (172.0, 48.9)
- added R29: 47k, Resistor_SMD:R_0603_1608Metric_Pad1.05x0.95mm_HandSolder, F.Cu at (172.0, 51.4)
- added R3: 4.7k, Resistor_SMD:R_0603_1608Metric_Pad1.05x0.95mm_HandSolder, F.Cu at (140.6, 77.0)
- added R30: 10k, Resistor_SMD:R_0603_1608Metric_Pad1.05x0.95mm_HandSolder, F.Cu at (167.6, 45.2)
- added R31: 100, Resistor_SMD:R_0603_1608Metric_Pad1.05x0.95mm_HandSolder, F.Cu at (173.2, 43.9)
- added R32: 100, Resistor_SMD:R_0603_1608Metric_Pad1.05x0.95mm_HandSolder, F.Cu at (163.3, 46.2)
- added R33: 330, Resistor_SMD:R_0603_1608Metric_Pad1.05x0.95mm_HandSolder, F.Cu at (163.3, 43.7)
- added R34: 5m, Resistor_SMD:R_2512_6332Metric, F.Cu at (160.8, 40.0)
- added R35: R, Resistor_SMD:R_0603_1608Metric_Pad1.05x0.95mm_HandSolder, F.Cu at (139.7, 53.6)
- added R36: R, Resistor_SMD:R_0603_1608Metric_Pad1.05x0.95mm_HandSolder, F.Cu at (135.3, 55.1)
- added R37: R, Resistor_SMD:R_0603_1608Metric_Pad1.05x0.95mm_HandSolder, F.Cu at (135.3, 57.6)
- added R38: 1.5k, Resistor_SMD:R_0603_1608Metric_Pad1.05x0.95mm_HandSolder, F.Cu at (141.9, 51.0)
- added R39: 68, Resistor_SMD:R_0603_1608Metric_Pad1.05x0.95mm_HandSolder, F.Cu at (128.7, 62.7)
- added R4: 10k, Resistor_SMD:R_0603_1608Metric_Pad1.05x0.95mm_HandSolder, F.Cu at (135.8, 85.2)
- added R40: 68, Resistor_SMD:R_0603_1608Metric_Pad1.05x0.95mm_HandSolder, F.Cu at (130.7, 60.2)
- added R41: R, Resistor_SMD:R_0603_1608Metric_Pad1.05x0.95mm_HandSolder, F.Cu at (124.4, 66.9)
- added R42: R, Resistor_SMD:R_0603_1608Metric_Pad1.05x0.95mm_HandSolder, F.Cu at (140.1, 84.5)
- added R43: R, Resistor_SMD:R_0603_1608Metric_Pad1.05x0.95mm_HandSolder, F.Cu at (104.7, 80.5)
- added R44: R, Resistor_SMD:R_0603_1608Metric_Pad1.05x0.95mm_HandSolder, F.Cu at (162.8, 50.9)
- added R5: 10k, Resistor_SMD:R_0603_1608Metric_Pad1.05x0.95mm_HandSolder, F.Cu at (140.6, 79.5)
- added R6: 5.23k, Resistor_SMD:R_0603_1608Metric_Pad1.05x0.95mm_HandSolder, F.Cu at (146.1, 75.6)
- added R7: 47k, Resistor_SMD:R_0603_1608Metric_Pad1.05x0.95mm_HandSolder, F.Cu at (136.2, 80.5)
- added R8: 10k, Resistor_SMD:R_0603_1608Metric_Pad1.05x0.95mm_HandSolder, F.Cu at (140.6, 82.0)
- added R9: 100, Resistor_SMD:R_0603_1608Metric_Pad1.05x0.95mm_HandSolder, F.Cu at (144.5, 84.5)
- added SW1: Function, Button_Switch_THT:SW_DIP_SPSTx04_Slide_9.78x12.34mm_W7.62mm_P2.54mm, F.Cu at (114.2, 40.8)
- added U1: LD1117S33TR_SOT223, Package_TO_SOT_SMD:SOT-223-3_TabPin2, F.Cu at (114.8, 111.3)
- added U2: ATmega644P-20AU, Package_QFP:TQFP-44_10x10mm_P0.8mm, F.Cu at (105.1, 44.8)
- added U3: OPA333xxDCK, Package_TO_SOT_SMD:SOT-353_SC-70-5_Handsoldering, F.Cu at (141.0, 73.8)
- added U4: OPA333xxDCK, Package_TO_SOT_SMD:SOT-353_SC-70-5_Handsoldering, F.Cu at (109.4, 73.8)
- added U5: OPA333xxDCK, Package_TO_SOT_SMD:SOT-353_SC-70-5_Handsoldering, F.Cu at (168.1, 39.5)
- added Y1: 12MHz, Crystal:Crystal_SMD_5032-4Pin_5.0x3.2mm, F.Cu at (113.4, 65.6)
Other:
- copper layers 0 -> 2
- net class Default added: clearance 0.2, trace_width 0.25, via_dia 0.8, via_drill 0.4
