File: leg-controller.sch (KiCad schematic (older format))
At the start: 34 parts, among them J1 Power, J12 UART, J13 USB_B_Mini, J14 ISP, J15 Motor_E, J16 Motor_D, J17 Motor_F, J2 I2C, SW1 Function, U1 LD1117S33TR_SOT223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

Commit message: Assigned remaining footprints
Parts:
- removed C2: CP, symbol Device:CP
- removed FB1: Ferrite_Bead, symbol Device:Ferrite_Bead
- removed R1: 0, Resistor_SMD:R_0603_1608Metric_Pad1.05x0.95mm_HandSolder, symbol Device:R
- added C2: 100n, Capacitor_SMD:C_0603_1608Metric_Pad1.08x0.95mm_HandSolder, symbol Device:C
- added NT1, NT2: Net-Tie_2, NetTie:NetTie-2_THT_Pad1.0mm, symbol Device:Net-Tie_2
- C1: footprint (none) -> Capacitor_THT:CP_Radial_D10.0mm_P5.00mm
- C3: value CP -> 10u; footprint (none) -> Capacitor_THT:CP_Radial_D5.0mm_P2.00mm
- D6: footprint (none) -> Diode_SMD:D_SOD-123F
- J12: footprint (none) -> Connector_PinHeader_2.54mm:PinHeader_1x04_P2.54mm_Vertical
- J13: footprint (none) -> Connector_USB:USB_Mini-B_Wuerth_65100516121_Horizontal
- J14: footprint (none) -> Connector_PinHeader_2.54mm:PinHeader_2x03_P2.54mm_Vertical
- SW1: footprint (none) -> Button_Switch_THT:SW_DIP_SPSTx04_Slide_9.78x12.34mm_W7.62mm_P2.54mm
- Y1: footprint (none) -> Crystal:Crystal_SMD_5032-4Pin_5.0x3.2mm
Connections:
- net +3.3VA: now also NT2.2
- net +3V3: now also NT2.1
- net +8V: now also C2.1
- net GND: now also C2.2, NT1.2
- net GNDPWR: now also NT1.1
Changed lines of the file:
@@
 EESchema Schematic File Version 4
-LIBS:leg-controller-cache
-EELAYER 29 0
+EELAYER 30 0
 EELAYER END
 $Descr A4 11693 8268
@@
 $EndComp
 $Comp
-L Device:Ferrite_Bead FB1
-U 1 1 6179AC46
-P 1200 1950
-F 0 "FB1" V 926 1950 50  0000 C CNN
-F 1 "Ferrite_Bead" V 1017 1950 50  0000 C CNN
-F 2 "" V 1130 1950 50  0001 C CNN
-F 3 "~" H 1200 1950 50  0001 C CNN
-	1    1200 1950
-	0    1    1    0
-$EndComp
-$Comp
 L power:GNDPWR #PWR01
 U 1 1 6179E286
@@
 F 0 "C1" H 1465 1146 50  0000 L CNN
 F 1 "470u" H 1465 1055 50  0000 L CNN
-F 2 "" H 1388 950 50  0001 C CNN
+F 2 "Capacitor_THT:CP_Radial_D10.0mm_P5.00mm" H 1388 950 50  0001 C CNN
 F 3 "~" H 1350 1100 50  0001 C CNN
 	1    1350 1100
@@
 $EndComp
 $Comp
-L Device:CP C2
-U 1 1 619318B9
-P 2350 1700
-F 0 "C2" H 2468 1746 50  0000 L CNN
-F 1 "CP" H 2468 1655 50  0000 L CNN
-F 2 "" H 2388 1550 50  0001 C CNN
-F 3 "~" H 2350 1700 50  0001 C CNN
-	1    2350 1700
-	1    0    0    -1
-$EndComp
-$Comp
 L Device:CP C3
 U 1 1 61932BEC
 P 3550 1700
 F 0 "C3" H 3668 1746 50  0000 L CNN
-F 1 "CP" H 3668 1655 50  0000 L CNN
-F 2 "" H 3588 1550 50  0001 C CNN
+F 1 "10u" H 3668 1655 50  0000 L CNN
+F 2 "Capacitor_THT:CP_Radial_D5.0mm_P2.00mm" H 3588 1550 50  0001 C CNN
 F 3 "~" H 3550 1700 50  0001 C CNN
 	1    3550 1700
@@
 F 0 "J14" H 2900 3567 50  0000 C CNN
 F 1 "ISP" H 2900 3476 50  0000 C CNN
-F 2 "" H 2850 3250 50  0001 C CNN
+F 2 "Connector_PinHeader_2.54mm:PinHeader_2x03_P2.54mm_Vertical" H 2850 3250 50  0001 C CNN
 F 3 "~" H 2850 3250 50  0001 C CNN
 	1    2850 3250
@@
 F 0 "D6" V 2146 1120 50  0000 R CNN
 F 1 "D" V 2055 1120 50  0000 R CNN
-F 2 "" H 2100 1200 50  0001 C CNN
+F 2 "Diode_SMD:D_SOD-123F" H 2100 1200 50  0001 C CNN
 F 3 "~" H 2100 1200 50  0001 C CNN
 	1    2100 1200
@@
 F 0 "J12" H 768 3517 50  0000 C CNN
 F 1 "UART" H 768 3426 50  0000 C CNN
-F 2 "" H 850 3200 50  0001 C CNN
+F 2 "Connector_PinHeader_2.54mm:PinHeader_1x04_P2.54mm_Vertical" H 850 3200 50  0001 C CNN
 F 3 "~" H 850 3200 50  0001 C CNN
 	1    850  3200
@@
 F 0 "Y1" H 4500 2432 50  0000 C CNN
 F 1 "12MHz" H 4500 2523 50  0000 C CNN
-F 2 "" H 4500 2700 50  0001 C CNN
+F 2 "Crystal:Crystal_SMD_5032-4Pin_5.0x3.2mm" H 4500 2700 50  0001 C CNN
 F 3 "~" H 4500 2700 50  0001 C CNN
 	1    4500 2700
@@
 Text GLabel 6750 4800 2    50   Input ~ 0
 ROT_DAT_C
-$Comp
-L Device:R R1
-U 1 1 619845E3
-P 5950 1800
-F 0 "R1" V 5743 1800 50  0000 C CNN
-F 1 "0" V 5834 1800 50  0000 C CNN
-F 2 "Resistor_SMD:R_0603_1608Metric_Pad1.05x0.95mm_HandSolder" V 5880 1800 50  0001 C CNN
-F 3 "~" H 5950 1800 50  0001 C CNN
-	1    5950 1800
-	0    1    1    0
-$EndComp
 Wire Wire Line
 	5700 1650 5700 1800
-Wire Wire Line
-	5700 1800 5800 1800
 Wire Wire Line
 	5700 1800 5700 1900
@@
 Wire Wire Line
 	6200 1900 6200 1800
-Wire Wire Line
-	6100 1800 6200 1800
 Connection ~ 6200 1800
 Wire Wire Line
@@
 F 0 "J13" H 2507 5267 50  0000 C CNN
 F 1 "USB_B_Mini" H 2507 5176 50  0000 C CNN
-F 2 "" H 2600 4750 50  0001 C CNN
+F 2 "Connector_USB:USB_Mini-B_Wuerth_65100516121_Horizontal" H 2600 4750 50  0001 C CNN
 F 3 "~" H 2600 4750 50  0001 C CNN
 	1    2450 4800
@@
 F 0 "SW1" H 1600 4767 50  0000 C CNN
 F 1 "Function" H 1600 4676 50  0000 C CNN
-F 2 "" H 1600 4300 50  0001 C CNN
+F 2 "Button_Switch_THT:SW_DIP_SPSTx04_Slide_9.78x12.34mm_W7.62mm_P2.54mm" H 1600 4300 50  0001 C CNN
 F 3 "~" H 1600 4300 50  0001 C CNN
 	1    1600 4300
 	1    0    0    -1
 $EndComp
+$Comp
+L Device:C C2
+U 1 1 6199BD38
+P 2350 1700
+F 0 "C2" H 2465 1746 50  0000 L CNN
+F 1 "100n" H 2465 1655 50  0000 L CNN
+F 2 "Capacitor_SMD:C_0603_1608Metric_Pad1.08x0.95mm_HandSolder" H 2388 1550 50  0001 C CNN
+F 3 "~" H 2350 1700 50  0001 C CNN
+	1    2350 1700
+	1    0    0    -1
+$EndComp
+$Comp
+L Device:Net-Tie_2 NT1
+U 1 1 619C0CF5
+P 1200 1950
+F 0 "NT1" H 1200 2131 50  0000 C CNN
+F 1 "Net-Tie_2" H 1200 2040 50  0000 C CNN
+F 2 "NetTie:NetTie-2_THT_Pad1.0mm" H 1200 1950 50  0001 C CNN
+F 3 "~" H 1200 1950 50  0001 C CNN
+	1    1200 1950
+	1    0    0    -1
+$EndComp
+Wire Wire Line
+	1100 1950 1050 1950
+Wire Wire Line
+	1300 1950 1350 1950
+$Comp
+L Device:Net-Tie_2 NT2
+U 1 1 619D7200
+P 5950 1800
+F 0 "NT2" H 5950 1981 50  0000 C CNN
+F 1 "Net-Tie_2" H 5950 1890 50  0000 C CNN
+F 2 "NetTie:NetTie-2_THT_Pad1.0mm" H 5950 1800 50  0001 C CNN
+F 3 "~" H 5950 1800 50  0001 C CNN
+	1    5950 1800
+	1    0    0    -1
+$EndComp
+Wire Wire Line
+	5700 1800 5850 1800
+Wire Wire Line
+	6050 1800 6200 1800
 $EndSCHEMATC

Commit message: Started workin on PCB layout. A bit faulty...
Parts:
- J15, J16, J17: footprint (none) -> Connector_PinHeader_2.54mm:PinHeader_1x05_P2.54mm_Vertical
- J2: footprint (none) -> Connector_PinHeader_2.54mm:PinHeader_1x03_P2.54mm_Vertical
Connections:
- no-connect marks 0 -> 3
Changed lines of the file:
@@
 EESchema Schematic File Version 4
-EELAYER 30 0
+LIBS:leg-controller-cache
+EELAYER 29 0
 EELAYER END
 $Descr A4 11693 8268
@@
 ROT_CLK_B
 Text GLabel 9250 2800 0    50   Input ~ 0
-ROT_CLK_DAT
+ROT_DAT_B
 Text GLabel 9250 3300 0    50   Input ~ 0
 MOTOR_C_CONTROL
@@
 F 0 "J15" H 9080 5692 50  0000 L CNN
 F 1 "Motor_E" H 9080 5601 50  0000 L CNN
-F 2 "" H 9000 5650 50  0001 C CNN
+F 2 "Connector_PinHeader_2.54mm:PinHeader_1x05_P2.54mm_Vertical" H 9000 5650 50  0001 C CNN
 F 3 "~" H 9000 5650 50  0001 C CNN
 	1    9000 5650
@@
 F 0 "J16" H 9730 4842 50  0000 L CNN
 F 1 "Motor_D" H 9730 4751 50  0000 L CNN
-F 2 "" H 9650 4800 50  0001 C CNN
+F 2 "Connector_PinHeader_2.54mm:PinHeader_1x05_P2.54mm_Vertical" H 9650 4800 50  0001 C CNN
 F 3 "~" H 9650 4800 50  0001 C CNN
 	1    9650 4800
@@
 F 0 "J17" H 10530 5692 50  0000 L CNN
 F 1 "Motor_F" H 10530 5601 50  0000 L CNN
-F 2 "" H 10450 5650 50  0001 C CNN
+F 2 "Connector_PinHeader_2.54mm:PinHeader_1x05_P2.54mm_Vertical" H 10450 5650 50  0001 C CNN
 F 3 "~" H 10450 5650 50  0001 C CNN
 	1    10450 5650
@@
 F 0 "J2" H 768 5417 50  0000 C CNN
 F 1 "I2C" H 768 5326 50  0000 C CNN
-F 2 "" H 850 5100 50  0001 C CNN
+F 2 "Connector_PinHeader_2.54mm:PinHeader_1x03_P2.54mm_Vertical" H 850 5100 50  0001 C CNN
 F 3 "~" H 850 5100 50  0001 C CNN
 	1    850  5100
@@
 Wire Wire Line
 	6050 1800 6200 1800
+$Comp
+L power:+3.3VA #PWR0125
+U 1 1 619A47FA
+P 4650 1200
+F 0 "#PWR0125" H 4650 1050 50  0001 C CNN
+F 1 "+3.3VA" H 4665 1373 50  0000 C CNN
+F 2 "" H 4650 1200 50  0001 C CNN
+F 3 "" H 4650 1200 50  0001 C CNN
+	1    4650 1200
+	1    0    0    -1
+$EndComp
+$Comp
+L power:PWR_FLAG #FLG0102
+U 1 1 619A4D22
+P 4650 1350
+F 0 "#FLG0102" H 4650 1425 50  0001 C CNN
+F 1 "PWR_FLAG" H 4650 1523 50  0000 C CNN
+F 2 "" H 4650 1350 50  0001 C CNN
+F 3 "~" H 4650 1350 50  0001 C CNN
+	1    4650 1350
+	-1   0    0    1
+$EndComp
+Wire Wire Line
+	4650 1200 4650 1350
+NoConn ~ 2350 5200
+NoConn ~ 2750 5000
+NoConn ~ 1300 4400
+$Comp
+L power:GNDPWR #PWR0124
+U 1 1 619D9FF3
+P 5000 1350
+AR Path="/619D9FF3" Ref="#PWR0124"  Part="1"
+AR Path="/619DAA4C/619D9FF3" Ref="#PWR?"  Part="1"
+AR Path="/61BE3D92/619D9FF3" Ref="#PWR?"  Part="1"
+AR Path="/618F2956/619D9FF3" Ref="#PWR?"  Part="1"
+AR Path="/618F4190/619D9FF3" Ref="#PWR?"  Part="1"
+F 0 "#PWR0124" H 5000 1150 50  0001 C CNN
+F 1 "GNDPWR" H 5004 1196 50  0000 C CNN
+F 2 "" H 5000 1300 50  0001 C CNN
+F 3 "" H 5000 1300 50  0001 C CNN
+	1    5000 1350
+	1    0    0    -1
+$EndComp
+$Comp
+L power:PWR_FLAG #FLG?
+U 1 1 619D9FF9
+P 5000 1200
+AR Path="/619DAA4C/619D9FF9" Ref="#FLG?"  Part="1"
+AR Path="/619D9FF9" Ref="#FLG0101"  Part="1"
+F 0 "#FLG0101" H 5000 1275 50  0001 C CNN
+F 1 "PWR_FLAG" H 5000 1373 50  0000 C CNN
+F 2 "" H 5000 1200 50  0001 C CNN
+F 3 "~" H 5000 1200 50  0001 C CNN
+	1    5000 1200
+	1    0    0    -1
+$EndComp
+Wire Wire Line
+	5000 1200 5000 1350
+$Comp
+L power:+8V #PWR0126
+U 1 1 619E96F8
+P 5300 1200
+AR Path="/619E96F8" Ref="#PWR0126"  Part="1"
+AR Path="/619DAA4C/619E96F8" Ref="#PWR?"  Part="1"
+AR Path="/61BE3D92/619E96F8" Ref="#PWR?"  Part="1"
+AR Path="/618F2956/619E96F8" Ref="#PWR?"  Part="1"
+AR Path="/618F4190/619E96F8" Ref="#PWR?"  Part="1"
+F 0 "#PWR0126" H 5300 1050 50  0001 C CNN
+F 1 "+8V" H 5315 1373 50  0000 C CNN
+F 2 "" H 5300 1200 50  0001 C CNN
+F 3 "" H 5300 1200 50  0001 C CNN
+	1    5300 1200
+	1    0    0    -1
+$EndComp
+$Comp
+L power:PWR_FLAG #FLG?
+U 1 1 619E96FE
+P 5300 1350
+AR Path="/619DAA4C/619E96FE" Ref="#FLG?"  Part="1"
+AR Path="/619E96FE" Ref="#FLG0103"  Part="1"
+F 0 "#FLG0103" H 5300 1425 50  0001 C CNN
+F 1 "PWR_FLAG" H 5300 1523 50  0000 C CNN
+F 2 "" H 5300 1350 50  0001 C CNN
+F 3 "~" H 5300 1350 50  0001 C CNN
+	1    5300 1350
+	-1   0    0    1
+$EndComp
+Wire Wire Line
+	5300 1350 5300 1200
 $EndSCHEMATC
