File: leg-controller.sch (KiCad schematic (older format))
At the start: 34 parts, among them J1 Power, J12 UART, J13 USB_B_Mini, J14 ISP, J15 Motor_E, J16 Motor_D, J17 Motor_F, J2 I2C, SW1 Function, U1 LD1117S33TR_SOT223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

Commit message: Placed components on the PCB
Parts:
- removed J12: UART, Connector_PinHeader_2.54mm:PinHeader_1x04_P2.54mm_Vertical, symbol Connector_Generic:Conn_01x04
- removed U2: ATmega644P-20AU, Package_QFP:TQFP-44_10x10mm_P0.8mm, symbol MCU_Microchip_ATmega:ATmega644P-20AU
- added U2: ATmega644P-20PU, Package_DIP:DIP-40_W15.24mm, symbol MCU_Microchip_ATmega:ATmega644P-20PU
- R35: value R -> 1.5k; footprint Resistor_SMD:R_0603_1608Metric_Pad1.05x0.95mm_HandSolder -> Resistor_SMD:R_0603_1608Metric
- R36, R37, R41: value R -> 330; footprint Resistor_SMD:R_0603_1608Metric_Pad1.05x0.95mm_HandSolder -> Resistor_SMD:R_0603_1608Metric
- R38, R39, R40: footprint Resistor_SMD:R_0603_1608Metric_Pad1.05x0.95mm_HandSolder -> Resistor_SMD:R_0603_1608Metric
Connections:
- net +3.3VA: now also U2.30 (AVCC)
- net +3V3: now also U2.10 (VCC)
- net FUNCTION_0: now also U2.37 (PA3)
- net FUNCTION_1: now also U2.36 (PA4)
- net GND: now also U2.11 (GND), U2.31 (GND)
- net I2C_SCL: now also U2.22 (PC0)
- net I2C_SDA: now also U2.23 (PC1)
- net LED_ERR: now also U2.2 (PB1)
- net LED_RUN: now also U2.1 (PB0)
- net MOTOR_A_CONTROL: now also U2.5 (PB4)
- net MOTOR_A_DISCONNECT: now also U2.24 (PC2)
- net MOTOR_A_SENSE: now also U2.40 (PA0)
- net MOTOR_B_CONTROL: now also U2.20 (PD6)
- net MOTOR_B_DISCONNECT: now also U2.25 (PC3)
- net MOTOR_B_SENSE: now also U2.39 (PA1)
- net MOTOR_C_CONTROL: now also U2.21 (PD7)
- net MOTOR_C_DISCONNECT: now also U2.26 (PC4)
- net MOTOR_C_SENSE: now also U2.38 (PA2)
- net RESET: now also SW1.4, U2.9 (~RESET)
- net ROT_CLK_A: now also U2.34 (PA6)
- net ROT_CLK_B: now also U2.14 (PD0)
- net ROT_CLK_C: now also U2.28 (PC6)
- net ROT_DAT_A: now also U2.33 (PA7)
- net ROT_DAT_B: now also U2.15 (PD1)
- net ROT_DAT_C: now also U2.29 (PC7)
- net SPI_MISO: now also U2.7 (PB6)
- net SPI_MOSI: now also U2.6 (PB5)
- net SPI_SCK: now also U2.8 (PB7)
- net SPI_SS_D: now also U2.27 (PC5)
- net SPI_SS_E: now also U2.18 (PD4)
- net SPI_SS_F: now also U2.19 (PD5)
- net USB_D+: now also U2.3 (PB2)
- net USB_D-: now also U2.4 (PB3)
- net at C6.1: now also U2.32 (AREF)
- net at C5.1, Y1.1: now also U2.12 (XTAL2)
- net at C4.1, Y1.2: now also U2.13 (XTAL1)
- net FUNCTION_2: no longer names the net of SW1.3
- new net LIMIT_SWITCH_A: U2.35 (PA5)
- new net LIMIT_SWITCH_B: U2.16 (PD2)
- new net LIMIT_SWITCH_C: U2.17 (PD3)
